File: pcb/effectpedal/ui.kicad_sch (KiCad schematic)
At the start: 120 parts

Commit message: Made progress on the PCB
Parts:
- removed J?: Conn_01x10_Male, symbol Connector:Conn_01x10_Male
- removed J? (x2): Conn_01x06_Male, symbol Connector:Conn_01x06_Male
- removed TP? (x20): TestPoint, symbol Connector:TestPoint
- added J12: Conn_01x16_Male, Connector_PinHeader_2.54mm:PinHeader_1x16_P2.54mm_Vertical, symbol Connector:Conn_01x16_Male
- added J17: Conn_01x06_Male, Connector_PinHeader_2.54mm:PinHeader_1x06_P2.54mm_Vertical, symbol Connector:Conn_01x06_Male
- added JP45: SolderJumper_2_Bridged, Jumper:SolderJumper-2_P1.3mm_Bridged2Bar_Pad1.0x1.5mm, symbol Jumper:SolderJumper_2_Bridged
- added JP46: SolderJumper_2_Open, Jumper:SolderJumper-2_P1.3mm_Open_Pad1.0x1.5mm, symbol Jumper:SolderJumper_2_Open
- C14, C15, C16: renamed from C?; footprint (none) -> Capacitor_SMD:C_0805_2012Metric
- D10, D11, D12, D13, D14, D15, D16, D5, D6, D7, D8, D9: renamed from D?; footprint (none) -> LED_SMD:LED_0805_2012Metric
- IC2, IC3, IC4: renamed from IC?; footprint QFN50P500X500X60-33N-D -> footprints:QFN50P500X500X60-33N-D
- J13, J14, J18: renamed from J?; footprint (none) -> Connector_PinHeader_2.54mm:PinHeader_1x06_P2.54mm_Vertical
- J15: renamed from J?; footprint (none) -> Connector_PinHeader_2.54mm:PinHeader_1x04_P2.54mm_Vertical
- JP33, JP34, JP36, JP37, JP38, JP39, JP41, JP42, JP44: renamed from JP?; footprint (none) -> Jumper:SolderJumper-2_P1.3mm_Open_Pad1.0x1.5mm
- JP35, JP40, JP43: renamed from JP?; footprint (none) -> Jumper:SolderJumper-2_P1.3mm_Bridged2Bar_Pad1.0x1.5mm
- R12, R13, R14, R15, R16, R17, R18, R19, R20, R21, R22, R23: renamed from R?; footprint (none) -> Resistor_SMD:R_0805_2012Metric
- RV1, RV2, RV3: renamed from RV?; footprint (none) -> footprints:PTV09A4015FB103
- S1, S10, S11, S12, S13, S14, S15, S16, S17, S18, S19, S2, S20, S21, S22, S23, S24, S25, S26, S27, S28, S29, S3, S30, S31, S32, S33, S34, S35, S36, S37, S38, S4, S5, S6, S7, S8, S9: renamed from S?; footprint SW-T3-2B-A-A3-S1 -> footprints:SW-T3-2B-A-A3-S1
- S39, S40: renamed from S?; footprint SS14D0839VG5PA -> footprints:SS14D0839VG5PA
- SW1, SW2, SW3, SW4, SW5, SW6, SW7, SW8: renamed from SW?; footprint (none) -> footprints:PTS810SJG250SMTRLFS
Connections:
- net GND1: now also SW2.1 (A), SW4.1 (A), SW6.1 (A), SW8.1 (A), J12.1 (Pin_1), J17.1 (Pin_1), J17.2 (Pin_2), J17.3 (Pin_3); no longer J13.2 (Pin_2), J13.3 (Pin_3), J14.2 (Pin_2), J14.4 (Pin_4), RV1.3, RV2.3, RV3.3
- net UI_3V3: now also J12.16 (Pin_16), J17.4 (Pin_4), J17.5 (Pin_5), J17.6 (Pin_6), JP46.2 (B); no longer J13.4 (Pin_4), J13.5 (Pin_5)
- net UI_RST: now also JP45.2 (B); no longer J18.5 (Pin_5)
- net UI_SCL: now also J12.7 (Pin_7)
- net UI_SDA: now also J12.6 (Pin_6)
- net at IC2.1 (P0_0): now also J12.8 (Pin_8)
- net at IC2.2 (P0_1): now also J12.9 (Pin_9)
- net at IC2.3 (P0_2): now also J12.10 (Pin_10)
- net at IC2.4 (P0_3): now also J12.11 (Pin_11)
- net at IC2.5 (P0_4): now also J12.12 (Pin_12)
- net at IC2.6 (P0_5): now also J12.13 (Pin_13)
- net at IC2.7 (P0_6): now also J12.14 (Pin_14)
- net at IC2.8 (P0_7): now also J12.15 (Pin_15)
- net at S1.1: now also IC3.9 (P1_0)
- net at S1.3: no longer IC3.9 (P1_0)
- new net: J18.5 (Pin_5), JP45.1 (A), JP46.1 (A)
- new net UI_AGND: J14.2 (Pin_2), J14.4 (Pin_4), RV1.3, RV2.3, RV3.3
- new net UI_EX1: J12.2 (Pin_2), J13.3 (Pin_3)
- new net UI_EX2: J12.3 (Pin_3), J13.4 (Pin_4)
- new net UI_EX3: J12.4 (Pin_4), J13.2 (Pin_2)
- new net UI_EX4: J12.5 (Pin_5), J13.5 (Pin_5)
- no-connect marks 0 -> 40
Other:
- note added: "Addr select"
- note added: "Expansion header"
- note added: "Hole in copper and soldermask for LED strip to shine through"
- note added: "Lower-right inter-board connector"
- note added: "OP-SEL LEDs"
- note added: "OP-SEL Switches"
- note removed: "Extra test points"
- note removed: "Lowerright inter-board connector"
- company: (none) -> Anton Liakhovitch
- title: (none) -> CRONCH UI Board
- moved on the sheet: C16, D10, D11, D12, D13, D14, D15, D16, D9, IC4, J13, J14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

Commit message: Mostly finished PCB
Parts:
- C14, C15, C16: Digikey Part Number (none) -> 478-1395-2-ND; Digikey Price/Stock (none) -> https://www.digikey.com/en/products/detail/kyocera-avx/0805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; MANUFACTURER (none) -> KYOCERA AVX; MPN (none) -> 08055C104KAT2A; Manufacturer_Name (none) -> KYOCERA AVX; Manufacturer_Part_Number (none) -> 08055C104KAT2A
- D10, D11, D12, D13, D14, D15, D16, D5, D6, D7, D8, D9: value LED -> LED, orange; Digikey Part Number (none) -> 2679-CTL0805FOG1TTR-ND; Digikey Price/Stock (none) -> https://www.digikey.com/en/products/detail/venkel/CTL0805FO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; MANUFACTURER (none) -> Venkel; MPN (none) -> CTL0805FOG1T; Manufacturer_Name (none) -> Venkel; Manufacturer_Part_Number (none) -> CTL0805FOG1T
- IC2, IC3, IC4: Digikey Part Number (none) -> 568-12879-2-ND; Digikey Price/Stock (none) -> https://www.digikey.com/en/products/detail/nxp-usa-inc/PCAL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; MANUFACTURER (none) -> NXP; MPN (none) -> PCAL6524HEAZ
- R12, R13, R14, R15, R16, R17, R18, R19, R20, R21, R22, R23: Digikey Part Number (none) -> 311-150CRTR-ND; Digikey Price/Stock (none) -> https://www.digikey.com/en/products/detail/yageo/RC0805FR-0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; MANUFACTURER (none) -> YAGEO; MPN (none) -> RC0805FR-07150RL; Manufacturer_Name (none) -> YAGEO; Manufacturer_Part_Number (none) -> RC0805FR-07150RL
- RV1, RV2, RV3: Digikey Part Number (none) -> PTV09A-4015F-B103-ND; Digikey Price/Stock (none) -> https://www.digikey.com/en/products/detail/bourns-inc/PTV09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; MANUFACTURER (none) -> Bourns Inc.; MPN (none) -> PTV09A-4015F-B103; Manufacturer_Name (none) -> Bourns Inc.; Manufacturer_Part_Number (none) -> PTV09A-4015F-B103
- S1, S10, S11, S12, S13, S14, S15, S16, S17, S18, S19, S2, S20, S21, S22, S23, S24, S25, S26, S27, S28, S29, S3, S30, S31, S32, S33, S34, S35, S36, S37, S38, S4, S5, S6, S7, S8, S9: Digikey Part Number (none) -> 2057-SW-T3-2B-A-A3-S1-ND; Digikey Price/Stock (none) -> https://www.digikey.com/en/products/detail/adam-tech/SW-T3-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; MANUFACTURER E-switch -> Adam Tech; MPN (none) -> SW-T3-2B-A-A3-S1; Manufacturer_Name (none) -> Adam Tech; Manufacturer_Part_Number (none) -> SW-T3-2B-A-A3-S1; STANDARD Manufacturer Recommendations -> (none)
- S39, S40: Digikey Part Number (none) -> CKN10727-ND; Digikey Price/Stock (none) -> https://www.digikey.com/en/products/detail/c-k/SS-14D0839-V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; MANUFACTURER (none) -> C & K COMPONENTS; MPN (none) -> SS14D0839VG5PA
- SW1, SW2, SW3, SW4, SW5, SW6, SW7, SW8: Digikey Part Number (none) -> CKN10504TR-ND; Digikey Price/Stock (none) -> https://www.digikey.com/en/products/detail/c-k/PTS810-SJG-2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; MANUFACTURER (none) -> C & K COMPONENTS; MPN (none) -> PTS810 SJG 250 SMTR LFS; Manufacturer_Name (none) -> C & K COMPONENTS; Manufacturer_Part_Number (none) -> PTS810 SJG 250 SMTR LFS
